File: pcb_bituhr/pcb_bituhr.kicad_sch (KiCad schematic)
At the start: 0 parts

Commit message: pico added
Parts:
- added A1: RaspberryPi_Pico, Module:RaspberryPi_Pico_Common_Unspecified, symbol MCU_Module:RaspberryPi_Pico
Connections:
- new net +3V3: A1.36 (3V3)
- new net +5V: A1.39 (VSYS)
- new net GND: A1.13 (GND), A1.18 (GND), A1.23 (GND), A1.28 (GND), A1.3 (GND), A1.38 (GND), A1.8 (GND)

Commit message: rtc und neopixel hinzugefügt
Parts:
- added DS3231: SCL, OptoDevice:Osram_DIL2_4.3x4.65mm_P5.08mm, symbol Connector:Conn_01x04_Pin
- added Neopixel1, Neopixel2, Neopixel3: Conn_01x03_Pin, OptoDevice:Osram_DIL2_4.3x4.65mm_P5.08mm, symbol Connector:Conn_01x03_Pin
Connections:
- net GND: now also DS3231.4 (Pin_4), Neopixel1.1 (Pin_1), Neopixel2.1 (Pin_1), Neopixel3.1 (Pin_1)
- net +3V3 renamed 3V3
- net 3V3: now also DS3231.3 (Pin_3), Neopixel1.3 (Pin_3), Neopixel2.3 (Pin_3), Neopixel3.3 (Pin_3)
- net +5V renamed 5V
- new net Neo1: Neopixel1.2 (Pin_2)
- new net Neo2: Neopixel2.2 (Pin_2)
- new net Neo3: Neopixel3.2 (Pin_2)
- new net SCL: DS3231.1 (Pin_1)
- new net SDA: DS3231.2 (Pin_2)

Commit message: do power supply properly
Connections:
- net 3V3: no longer DS3231.3 (Pin_3), Neopixel1.3 (Pin_3), Neopixel2.3 (Pin_3), Neopixel3.3 (Pin_3)
- new net +3V3: DS3231.3 (Pin_3), Neopixel1.3 (Pin_3), Neopixel2.3 (Pin_3), Neopixel3.3 (Pin_3)

Commit message: add all componets
Parts:
- added Button, Potentiometer: Conn_01x03_Pin, OptoDevice:Osram_DIL2_4.3x4.65mm_P5.08mm, symbol Connector:Conn_01x03_Pin
- added Kippschalter1, Kippschalter2: Conn_01x02_Pin, symbol Connector:Conn_01x02_Pin
- added PowerIN: Screw_Terminal_01x02, Connector_Audio:Jack_speakON_Neutrik_NL4MDXX-H-2_Horizontal, symbol Connector:Screw_Terminal_01x02
Connections:
- net +3V3: now also Button.3 (Pin_3), Kippschalter1.1 (Pin_1), Kippschalter2.1 (Pin_1), Potentiometer.3 (Pin_3)
- net GND: now also Button.1 (Pin_1), Potentiometer.1 (Pin_1), PowerIN.2 (Pin_2)
- net Potentiometer: now reaches A1.31 (GPIO26_ADC0)
- net Potentiometer: now also Potentiometer.2 (Pin_2)
- new net +5V: PowerIN.1 (Pin_1)
- new net Button: Button.2 (Pin_2)
- new net Kipp1: Kippschalter1.2 (Pin_2)
- new net Kipp2: Kippschalter2.2 (Pin_2)
Other:
- moved on the sheet: DS3231, Neopixel1, Neopixel2, Neopixel3

Commit message: add all componet
Connections:
- net 3V3 is gone; now on net +3V3: A1.36 (3V3)
- net 5V is gone; now on net +5V: A1.39 (VSYS)
- net Button: now also A1.29 (GPIO22)
- net Kipp1: now also A1.26 (GPIO20)
- net Kipp2: now also A1.27 (GPIO21)
- net Neo1: now also A1.4 (GPIO2)
- net Neo2: now also A1.5 (GPIO3)
- net Neo3: now also A1.6 (GPIO4)
- net SCL: now also A1.22 (GPIO17)
- net SDA: now also A1.21 (GPIO16)
Changed lines of the file:
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@@
+	(wire
+		(pts
+			(xy 167.64 93.98) (xy 172.72 93.98)
+		)
+		(stroke
+			(width 0)
+			(type default)
+		)
+	)
 	(wire
 		(pts
@@
 	(wire
 		(pts
+			(xy 167.64 83.82) (xy 172.72 83.82)
+		)
+		(stroke
+			(width 0)
+			(type default)
+		)
+	)
+	(wire
+		(pts
 			(xy 72.39 78.74) (xy 74.93 78.74)
 		)
@@
 	(wire
 		(pts
+			(xy 114.3 88.9) (xy 121.92 88.9)
+		)
+		(stroke
+			(width 0)
+			(type default)
+		)
+	)
+	(wire
+		(pts
+			(xy 167.64 99.06) (xy 172.72 99.06)
+		)
+		(stroke
+			(width 0)
+			(type default)
+		)
+	)
+	(wire
+		(pts
 			(xy 210.82 88.9) (xy 215.9 88.9)
 		)
@@
 	(wire
 		(pts
+			(xy 167.64 96.52) (xy 172.72 96.52)
+		)
+		(stroke
+			(width 0)
+			(type default)
+		)
+	)
+	(wire
+		(pts
 			(xy 210.82 104.14) (xy 215.9 104.14)
 		)
@@
 	(wire
 		(pts
+			(xy 114.3 91.44) (xy 121.92 91.44)
+		)
+		(stroke
+			(width 0)
+			(type default)
+		)
+	)
+	(wire
+		(pts
 			(xy 167.64 109.22) (xy 171.45 109.22)
 		)
@@
 	(wire
 		(pts
+			(xy 114.3 86.36) (xy 121.92 86.36)
+		)
+		(stroke
+			(width 0)
+			(type default)
+		)
+	)
+	(wire
+		(pts
 			(xy 73.66 109.22) (xy 76.2 109.22)
 		)
@@
 		(pts
 			(xy 73.66 106.68) (xy 76.2 106.68)
+		)
+		(stroke
+			(width 0)
+			(type default)
+		)
+	)
+	(wire
+		(pts
+			(xy 167.64 86.36) (xy 172.72 86.36)
 		)
 		(stroke
@@
 		)
 	)
+	(label "Button"
+		(at 172.72 99.06 0)
+		(effects
+			(font
+				(size 1.27 1.27)
+			)
+			(justify left bottom)
+		)
+	)
 	(label "Neo1"
 		(at 210.82 72.39 0)
@@
 		)
 	)
+	(label "SDA"
+		(at 172.72 83.82 0)
+		(effects
+			(font
+				(size 1.27 1.27)
+			)
+			(justify left bottom)
+		)
+	)
 	(label "Potentiometer"
 		(at 203.2 120.65 0)
@@
 		)
 	)
+	(label "Neo1"
+		(at 114.3 86.36 180)
+		(effects
+			(font
+				(size 1.27 1.27)
+			)
+			(justify right bottom)
+		)
+	)
 	(label "SCL"
 		(at 74.93 71.12 0)
@@
 		)
 	)
+	(label "SCL"
+		(at 172.72 86.36 0)
+		(effects
+			(font
+				(size 1.27 1.27)
+			)
+			(justify left bottom)
+		)
+	)
+	(label "Neo2"
+		(at 114.3 88.9 180)
+		(effects
+			(font
+				(size 1.27 1.27)
+			)
+			(justify right bottom)
+		)
+	)
 	(label "Button"
 		(at 78.74 121.92 0)
@@
 	(label "Neo3"
 		(at 210.82 101.6 0)
+		(effects
+			(font
+				(size 1.27 1.27)
+			)
+			(justify left bottom)
+		)
+	)
+	(label "Neo3"
+		(at 114.3 91.44 180)
+		(effects
+			(font
+				(size 1.27 1.27)
+			)
+			(justify right bottom)
+		)
+	)
+	(label "Kipp1"
+		(at 172.72 93.98 0)
+		(effects
+			(font
+				(size 1.27 1.27)
+			)
+			(justify left bottom)
+		)
+	)
+	(label "Kipp2"
+		(at 172.72 96.52 0)
 		(effects
 			(font
@@
 			)
 		)
-		(property "Value" "5V"
+		(property "Value" "+5V"
 			(at 139.7 50.8 0)
 			(show_name no)
@@
 			)
 		)
-		(property "Value" "3V3"
+		(property "Value" "+3V3"
 			(at 149.86 50.8 0)
 			(show_name no)

Commit message: finished scematic
Parts:
- DS3231: value SCL -> Conn_01x04_Pin; footprint OptoDevice:Osram_DIL2_4.3x4.65mm_P5.08mm -> Connector_PinSocket_2.54mm:PinSocket_1x04_P2.54mm_Vertical
- renumbered Button to Button1, Potentiometer to Potentiometer1, PowerIN to PowerIN1
Changed lines of the file:
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@@
 		(in_pos_files yes)
 		(dnp no)
-		(property "Reference" "Potentiometer"
+		(property "Reference" "Potentiometer1"
 			(at 218.44 113.792 0)
 			(show_name no)
@@
 			(project "pcb_bituhr"
 				(path "/d6c34df6-2d93-4be8-987b-02bf51a7e5d9"
-					(reference "Potentiometer")
+					(reference "Potentiometer1")
 					(unit 1)
 				)
@@
 			)
 		)
-		(property "Value" "SCL"
+		(property "Value" "Conn_01x04_Pin"
 			(at 67.945 68.58 0)
 			(hide yes)
@@
 			)
 		)
-		(property "Footprint" "OptoDevice:Osram_DIL2_4.3x4.65mm_P5.08mm"
+		(property "Footprint" "Connector_PinSocket_2.54mm:PinSocket_1x04_P2.54mm_Vertical"
 			(at 67.31 73.66 0)
 			(hide yes)
@@
 		(in_pos_files yes)
 		(dnp no)
-		(property "Reference" "Button"
+		(property "Reference" "Button1"
 			(at 73.152 116.84 0)
 			(show_name no)
@@
 			(project "pcb_bituhr"
 				(path "/d6c34df6-2d93-4be8-987b-02bf51a7e5d9"
-					(reference "Button")
+					(reference "Button1")
 					(unit 1)
 				)
@@
 		(dnp no)
 		(property "Reference" "Kippschalter2"
-			(at 72.39 102.108 0)
+			(at 72.898 102.87 0)
 			(show_name no)
 			(do_not_autoplace no)
@@
 		(dnp no)
 		(fields_autoplaced yes)
-		(property "Reference" "PowerIN"
+		(property "Reference" "PowerIN1"
 			(at 74.93 130.81 0)
 			(show_name no)
@@
 			(project "pcb_bituhr"
 				(path "/d6c34df6-2d93-4be8-987b-02bf51a7e5d9"
-					(reference "PowerIN")
-					(unit 1)
-				)
+					(reference "PowerIN1")
+					(unit 1)
+				)

Commit message: add fottprints
Parts:
- A1: footprint Module:RaspberryPi_Pico_Common_Unspecified -> Connector_JST:JST_PUD_B40B-PUDSS_2x20_P2.00mm_Vertical
- Button1, Neopixel1, Neopixel2, Neopixel3, Potentiometer1: footprint OptoDevice:Osram_DIL2_4.3x4.65mm_P5.08mm -> Connector_JST:JST_XH_B3B-XH-A_1x03_P2.50mm_Vertical
- Kippschalter1, Kippschalter2: footprint (none) -> Connector_JST:JST_XH_B2B-XH-A_1x02_P2.50mm_Vertical
- PowerIN1: footprint Connector_Audio:Jack_speakON_Neutrik_NL4MDXX-H-2_Horizontal -> TerminalBlock:TerminalBlock_Xinya_XY308-2.54-2P_1x02_P2.54mm_Horizontal
Changed lines of the file:
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@@
 			)
 		)
-		(property "Footprint" ""
+		(property "Footprint" "Connector_JST:JST_XH_B2B-XH-A_1x02_P2.50mm_Vertical"
 			(at 68.58 93.98 0)
 			(hide yes)
@@
 			)
 		)
-		(property "Footprint" "OptoDevice:Osram_DIL2_4.3x4.65mm_P5.08mm"
+		(property "Footprint" "Connector_JST:JST_XH_B3B-XH-A_1x03_P2.50mm_Vertical"
 			(at 220.98 101.6 0)
 			(hide yes)
@@
 			)
 		)
-		(property "Footprint" "OptoDevice:Osram_DIL2_4.3x4.65mm_P5.08mm"
+		(property "Footprint" "Connector_JST:JST_XH_B3B-XH-A_1x03_P2.50mm_Vertical"
 			(at 220.98 120.65 0)
 			(hide yes)
@@
 			)
 		)
-		(property "Footprint" "OptoDevice:Osram_DIL2_4.3x4.65mm_P5.08mm"
+		(property "Footprint" "Connector_JST:JST_XH_B3B-XH-A_1x03_P2.50mm_Vertical"
 			(at 220.98 72.39 0)
 			(hide yes)
@@
 			)
 		)
-		(property "Footprint" "OptoDevice:Osram_DIL2_4.3x4.65mm_P5.08mm"
+		(property "Footprint" "Connector_JST:JST_XH_B3B-XH-A_1x03_P2.50mm_Vertical"
 			(at 220.98 86.36 0)
 			(hide yes)
@@
 			)
 		)
-		(property "Footprint" "Module:RaspberryPi_Pico_Common_Unspecified"
+		(property "Footprint" "Connector_JST:JST_PUD_B40B-PUDSS_2x20_P2.00mm_Vertical"
 			(at 144.78 143.51 0)
 			(hide yes)
@@
 			)
 		)
-		(property "Footprint" "OptoDevice:Osram_DIL2_4.3x4.65mm_P5.08mm"
+		(property "Footprint" "Connector_JST:JST_XH_B3B-XH-A_1x03_P2.50mm_Vertical"
 			(at 71.12 121.92 0)
 			(hide yes)
@@
 			)
 		)
-		(property "Footprint" ""
+		(property "Footprint" "Connector_JST:JST_XH_B2B-XH-A_1x02_P2.50mm_Vertical"
 			(at 68.58 106.68 0)
 			(hide yes)
@@
 			)
 		)
-		(property "Footprint" "Connector_Audio:Jack_speakON_Neutrik_NL4MDXX-H-2_Horizontal"
+		(property "Footprint" "TerminalBlock:TerminalBlock_Xinya_XY308-2.54-2P_1x02_P2.54mm_Horizontal"
 			(at 74.93 137.16 0)
 			(hide yes)

Commit message: finisch scemetic
Parts:
- A1: footprint Connector_JST:JST_PUD_B40B-PUDSS_2x20_P2.00mm_Vertical -> Module:RaspberryPi_Pico_Common_THT
Changed lines of the file:
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@@
-	(wire
-		(pts
-			(xy 80.01 134.62) (xy 83.82 134.62)
-		)
-		(stroke
-			(width 0)
-			(type default)
-		)
-	)
 	(wire
 		(pts
@@
 	(wire
 		(pts
+			(xy 80.01 134.62) (xy 85.09 134.62)
+		)
+		(stroke
+			(width 0)
+			(type default)
+		)
+	)
+	(wire
+		(pts
 			(xy 167.64 96.52) (xy 172.72 96.52)
 		)
@@
 	(wire
 		(pts
-			(xy 80.01 137.16) (xy 83.82 137.16)
-		)
-		(stroke
-			(width 0)
-			(type default)
-		)
-	)
-	(wire
-		(pts
 			(xy 210.82 86.36) (xy 215.9 86.36)
 		)
@@
 		(pts
 			(xy 73.66 96.52) (xy 76.2 96.52)
+		)
+		(stroke
+			(width 0)
+			(type default)
+		)
+	)
+	(wire
+		(pts
+			(xy 80.01 137.16) (xy 85.09 137.16)
 		)
 		(stroke
@@
 	(symbol
 		(lib_id "power:+5V")
-		(at 83.82 137.16 270)
+		(at 85.09 137.16 270)
 		(unit 1)
 		(body_style 1)
@@
 		(in_pos_files yes)
 		(dnp no)
-		(fields_autoplaced yes)
 		(property "Reference" "#PWR018"
-			(at 80.01 137.16 0)
+			(at 81.28 137.16 0)
 			(hide yes)
 			(show_name no)
@@
 		)
 		(property "Value" "+5V"
-			(at 87.63 137.1599 90)
+			(at 88.646 137.16 90)
 			(show_name no)
 			(do_not_autoplace no)
@@
 		)
 		(property "Footprint" ""
-			(at 83.82 137.16 0)
+			(at 85.09 137.16 0)
 			(hide yes)
 			(show_name no)
@@
 		)
 		(property "Datasheet" ""
-			(at 83.82 137.16 0)
+			(at 85.09 137.16 0)
 			(hide yes)
 			(show_name no)
@@
 		)
 		(property "Description" "Power symbol creates a global label with name \"+5V\""
-			(at 83.82 137.16 0)
+			(at 85.09 137.16 0)
 			(hide yes)
 			(show_name no)
@@
 	(symbol
 		(lib_id "power:GND")
-		(at 83.82 134.62 90)
+		(at 85.09 134.62 90)
 		(unit 1)
 		(body_style 1)
@@
 		(fields_autoplaced yes)
 		(property "Reference" "#PWR019"
-			(at 90.17 134.62 0)
+			(at 91.44 134.62 0)
 			(hide yes)
 			(show_name no)
@@
 		)
 		(property "Value" "GND"
-			(at 87.63 134.6199 90)
+			(at 88.9 134.6199 90)
 			(show_name no)
 			(do_not_autoplace no)
@@
 		)
 		(property "Footprint" ""
-			(at 83.82 134.62 0)
+			(at 85.09 134.62 0)
 			(hide yes)
 			(show_name no)
@@
 		)
 		(property "Datasheet" ""
-			(at 83.82 134.62 0)
+			(at 85.09 134.62 0)
 			(hide yes)
 			(show_name no)
@@
 		)
 		(property "Description" "Power symbol creates a global label with name \"GND\" , ground"
-			(at 83.82 134.62 0)
+			(at 85.09 134.62 0)
 			(hide yes)
 			(show_name no)
@@
 			)
 		)
-		(property "Footprint" "Connector_JST:JST_PUD_B40B-PUDSS_2x20_P2.00mm_Vertical"
+		(property "Footprint" "Module:RaspberryPi_Pico_Common_THT"
 			(at 144.78 143.51 0)
 			(hide yes)
